Commit message: Update QUB humanoid to 13 DOF

File: resources/robots/QUB/urdf/QUB.urdf (robot description, URDF)
Before this commit: robot QUB, 28 links, 27 joints
Joints:
- joint L_Thigh_pitch_1_joint: axis -0.032631 0.99947 0 -> (none); limit lower=-1.57 upper=1.57 effort=30.0 velocity=5.0 -> (none); type revolute -> fixed
- joint L_Thigh_pitch_2_joint: axis 0.032631 -0.99947 0 -> (none); limit lower=-1.57 upper=1.57 effort=30.0 velocity=5.0 -> (none); type revolute -> fixed
- joint R_Thigh_pitch_1_joint: axis 0.0326305757533488 -0.999467480974746 0 -> (none); limit lower=-1.57 upper=1.57 effort=30.0 velocity=5.0 -> (none); type revolute -> fixed
- joint R_Thigh_pitch_2_joint: axis 0.0326305757533486 -0.999467480974746 0 -> (none); limit lower=-1.57 upper=1.57 effort=30.0 velocity=5.0 -> (none); type revolute -> fixed
